File: CH330.sch (KiCad schematic (older format))
At the start: 9 parts, among them J1 USB_B_Micro, J2 Conn_01x04_Female, U1 CH330

Commit message: add: update schematics to USB C
Parts:
- removed J1: USB_B_Micro, Connector_USB:USB_Micro-B_Molex_47346-0001, symbol Connector:USB_B_Micro
- added P1: USB_C_Plug_USB2.0, Connector_USB:USB_C_Receptacle_XKB_U262-16XN-4BVC11, symbol Connector:USB_C_Plug_USB2.0
- added R3, R4: 5.1k, Resistor_SMD:R_0603_1608Metric, symbol Device:R_Small
- U1: value CH330 -> CH330N; symbol otter:CH330 -> CH330-rescue:CH330-otter
Connections:
- net labels removed: D+, D-, RTS, RXD, TXD, V3
- wire segments 1 -> 33
- no-connect marks 0 -> 1
Other:
- moved on the sheet: C1, C2, D1, D2, J2, R1, R2

Commit message: add: BOM
Parts:
- C1, C2: Mfr. Part (none) -> CC0603KRX7R9BB104
- D1, D2: Mfr. Part (none) -> 19-217/R6C-AL1M2VY/3T
- P1: Mfr. Part (none) -> U262-161N-4BVC11
- R1, R2: Mfr. Part (none) -> 0603WAF2200T5E
- R3, R4: Mfr. Part (none) -> 0603WAJ0512T5E
- U1: Mfr. Part (none) -> CH330N
Changed lines of the file:
@@
 F 1 "CH330N" H 6100 4184 50  0000 C CNN
 F 2 "Package_SO:SOIC-8_3.9x4.9mm_P1.27mm" H 5950 3900 50  0001 C CNN
-F 3 "" H 5950 3900 50  0001 C CNN
+F 3 "https://datasheet.lcsc.com/szlcsc/2008191734_WCH-Jiangsu-Qin-Heng-CH330N_C108996.pdf" H 5950 3900 50  0001 C CNN
+F 4 "CH330N" H 6100 3900 50  0001 C CNN "Mfr. Part"
 	1    6100 3900
 	1    0    0    -1
@@
 F 1 "100n" H 6592 3405 50  0000 L CNN
 F 2 "Capacitor_SMD:C_0603_1608Metric" H 6500 3450 50  0001 C CNN
-F 3 "~" H 6500 3450 50  0001 C CNN
+F 3 "https://datasheet.lcsc.com/szlcsc/YAGEO-CC0603KRX7R9BB104_C14663.pdf" H 6500 3450 50  0001 C CNN
+F 4 "CC0603KRX7R9BB104" H 6500 3450 50  0001 C CNN "Mfr. Part"
 	1    6500 3450
 	-1   0    0    1
@@
 F 1 "100n" H 5692 3305 50  0000 L CNN
 F 2 "Capacitor_SMD:C_0603_1608Metric" H 5600 3350 50  0001 C CNN
-F 3 "~" H 5600 3350 50  0001 C CNN
+F 3 "https://datasheet.lcsc.com/szlcsc/YAGEO-CC0603KRX7R9BB104_C14663.pdf" H 5600 3350 50  0001 C CNN
+F 4 "CC0603KRX7R9BB104" H 5600 3350 50  0001 C CNN "Mfr. Part"
 	1    5600 3350
 	1    0    0    -1
@@
 F 1 "LED" V 6750 3300 50  0000 R CNN
 F 2 "LED_SMD:LED_0603_1608Metric" H 6800 3400 50  0001 C CNN
-F 3 "~" H 6800 3400 50  0001 C CNN
+F 3 "https://datasheet.lcsc.com/szlcsc/Everlight-Elec-19-217-R6C-AL1M2VY-3T_C72044.pdf" H 6800 3400 50  0001 C CNN
+F 4 "19-217/R6C-AL1M2VY/3T" H 6800 3400 50  0001 C CNN "Mfr. Part"
 	1    6800 3400
 	0    -1   -1   0
@@
 F 1 "220" H 6900 3600 50  0000 L CNN
 F 2 "Resistor_SMD:R_0603_1608Metric" H 6800 3650 50  0001 C CNN
-F 3 "~" H 6800 3650 50  0001 C CNN
+F 3 "https://datasheet.lcsc.com/szlcsc/Uniroyal-Elec-0603WAF2200T5E_C22962.pdf" H 6800 3650 50  0001 C CNN
+F 4 "0603WAF2200T5E" H 6800 3650 50  0001 C CNN "Mfr. Part"
 	1    6800 3650
 	1    0    0    -1
@@
 F 1 "220" H 7200 3600 50  0000 L CNN
 F 2 "Resistor_SMD:R_0603_1608Metric" H 7100 3650 50  0001 C CNN
-F 3 "~" H 7100 3650 50  0001 C CNN
+F 3 "https://datasheet.lcsc.com/szlcsc/Uniroyal-Elec-0603WAF2200T5E_C22962.pdf" H 7100 3650 50  0001 C CNN
+F 4 "0603WAF2200T5E" H 7100 3650 50  0001 C CNN "Mfr. Part"
 	1    7100 3650
 	1    0    0    -1
@@
 F 1 "USB_C_Plug_USB2.0" H 4707 4626 50  0000 C CNN
 F 2 "Connector_USB:USB_C_Receptacle_XKB_U262-16XN-4BVC11" H 4750 3850 50  0001 C CNN
-F 3 "https://www.usb.org/sites/default/files/documents/usb_type-c.zip" H 4750 3850 50  0001 C CNN
+F 3 "https://datasheet.lcsc.com/szlcsc/2002271811_XKB-Connectivity-U262-161N-4BVC11_C319148.pdf" H 4750 3850 50  0001 C CNN
+F 4 "U262-161N-4BVC11" H 4600 3850 50  0001 C CNN "Mfr. Part"
 	1    4600 3850
 	1    0    0    -1
@@
 F 1 "LED" V 7050 3300 50  0000 R CNN
 F 2 "LED_SMD:LED_0603_1608Metric" H 7100 3400 50  0001 C CNN
-F 3 "~" H 7100 3400 50  0001 C CNN
+F 3 "https://datasheet.lcsc.com/szlcsc/Everlight-Elec-19-217-R6C-AL1M2VY-3T_C72044.pdf" H 7100 3400 50  0001 C CNN
+F 4 "19-217/R6C-AL1M2VY/3T" H 7100 3400 50  0001 C CNN "Mfr. Part"
 	1    7100 3400
 	0    -1   -1   0
@@
 F 1 "5.1k" H 5450 3400 50  0000 L CNN
 F 2 "Resistor_SMD:R_0603_1608Metric" H 5400 3450 50  0001 C CNN
-F 3 "~" H 5400 3450 50  0001 C CNN
+F 3 "https://datasheet.lcsc.com/szlcsc/Uniroyal-Elec-0603WAJ0512T5E_C26000.pdf" H 5400 3450 50  0001 C CNN
+F 4 "0603WAJ0512T5E" H 5400 3450 50  0001 C CNN "Mfr. Part"
 	1    5400 3450
 	0    -1   -1   0
@@
 F 1 "5.1k" H 5200 3500 50  0000 L CNN
 F 2 "Resistor_SMD:R_0603_1608Metric" H 5400 3550 50  0001 C CNN
-F 3 "~" H 5400 3550 50  0001 C CNN
+F 3 "https://datasheet.lcsc.com/szlcsc/Uniroyal-Elec-0603WAJ0512T5E_C26000.pdf" H 5400 3550 50  0001 C CNN
+F 4 "0603WAJ0512T5E" H 5400 3550 50  0001 C CNN "Mfr. Part"
 	1    5400 3550
 	0    -1   -1   0
